File: PinCushion.kicad_sch (KiCad schematic)
At the start: 5 parts

Commit message: updates
Parts:
- added U6, U7, U8, U9, U? (x3): (no value), symbol symbols:PinLengths
Connections:
- net at U1.27 (Non_Logic): now also U3.1 (Line); no longer U3.2 (Line)
- net at U3.27 (Non_Logic): now also U5.1 (Line); no longer U5.2 (Line)
Other:
- note added: "Mirrored X"
- note added: "Mirrored Y"
- note added: "R0"
- note added: "R1"
- note added: "R2"
- note added: "R3"
Changed lines of the file:
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@@
     (stroke (width 0) (type default) (color 0 0 0 0))
+  )
+  (text "R3" (at 89.535 186.69 0)
+    (effects (font (size 1.27 1.27)) (justify left bottom))
+  )
+  (text "Mirrored X" (at 186.055 135.255 0)
+    (effects (font (size 1.27 1.27)) (justify left bottom))
+  )
+  (text "R1" (at 87.63 159.385 0)
+    (effects (font (size 1.27 1.27)) (justify left bottom))
+  )
+  (text "R2" (at 62.23 186.69 0)
+    (effects (font (size 1.27 1.27)) (justify left bottom))
+  )
+  (text "Mirrored Y" (at 221.615 158.75 0)
+    (effects (font (size 1.27 1.27)) (justify left bottom))
+  )
+  (text "R0" (at 61.595 163.195 0)
+    (effects (font (size 1.27 1.27)) (justify left bottom))
+  )
+  (symbol (lib_id "symbols:PinLengths") (at 194.945 149.86 0) (mirror x) (unit 1)
+    (in_bom yes) (on_board yes) (fields_autoplaced)
+    (property "Reference" "U?" (id 0) (at 191.135 160.02 0))
+    (property "Value" "" (id 1) (at 191.135 157.48 0))
+    (property "Footprint" "" (id 2) (at 182.88 161.29 0)
+      (effects (font (size 1.27 1.27)) hide)
+    )
+    (property "Datasheet" "" (id 3) (at 182.88 161.29 0)
+      (effects (font (size 1.27 1.27)) hide)
+    )
+    (pin "1")
+    (pin "2")
+    (pin "3")
+    (pin "4")
+    (pin "5")
+    (pin "6")
   )
   (symbol (lib_name "PinCushion_2") (lib_id "symbols:PinCushion") (at 144.78 40.64 0) (unit 1)
@@
       (effects (font (size 1.27 1.27)) hide)
     )
+    (pin "1")
     (pin "10")
     (pin "11")
@@
     (pin "19")
     (pin "2")
-    (pin "2")
     (pin "20")
     (pin "21")
@@
     (pin "9")
   )
+  (symbol (lib_name "PinLengths_1") (lib_id "symbols:PinLengths") (at 110.49 132.08 90) (unit 1)
+    (in_bom yes) (on_board yes) (fields_autoplaced)
+    (property "Reference" "U?" (id 0) (at 125.095 134.6199 90)
+      (effects (font (size 1.27 1.27)) (justify right))
+    )
+    (property "Value" "" (id 1) (at 125.095 137.1599 90)
+      (effects (font (size 1.27 1.27)) (justify right))
+    )
+    (property "Footprint" "" (id 2) (at 99.06 144.145 0)
+      (effects (font (size 1.27 1.27)) hide)
+    )
+    (property "Datasheet" "" (id 3) (at 99.06 144.145 0)
+      (effects (font (size 1.27 1.27)) hide)
+    )
+    (pin "1")
+    (pin "2")
+    (pin "3")
+    (pin "4")
+    (pin "5")
+    (pin "6")
+  )
   (symbol (lib_name "PinCushion_4") (lib_id "symbols:PinCushion") (at 71.12 104.14 0) (unit 1)
     (in_bom yes) (on_board yes) (fields_autoplaced)
@@
       (effects (font (size 1.27 1.27)) hide)
     )
+    (pin "1")
     (pin "10")
     (pin "11")
@@
     (pin "19")
     (pin "2")
-    (pin "2")
     (pin "20")
     (pin "21")
@@
       (effects (font (size 1.27 1.27)) hide)
     )
+    (pin "1")
     (pin "10")
     (pin "11")
@@
     (pin "19")
     (pin "2")
-    (pin "2")
     (pin "20")
     (pin "21")
@@
     (pin "9")
   )
+  (symbol (lib_id "symbols:PinLengths") (at 222.885 142.24 0) (mirror y) (unit 1)
+    (in_bom yes) (on_board yes) (fields_autoplaced)
+    (property "Reference" "U?" (id 0) (at 226.695 132.08 0))
+    (property "Value" "" (id 1) (at 226.695 134.62 0))
+    (property "Footprint" "" (id 2) (at 234.95 130.81 0)
+      (effects (font (size 1.27 1.27)) hide)
+    )
+    (property "Datasheet" "" (id 3) (at 234.95 130.81 0)
+      (effects (font (size 1.27 1.27)) hide)
+    )
+    (pin "1")
+    (pin "2")
+    (pin "3")
+    (pin "4")
+    (pin "5")
+    (pin "6")
+  )
   (symbol (lib_name "PinCushion_3") (lib_id "symbols:PinCushion") (at 213.36 104.14 0) (unit 1)
     (in_bom yes) (on_board yes) (fields_autoplaced)
@@
       (effects (font (size 1.27 1.27)) hide)
     )
+    (pin "1")
     (pin "10")
     (pin "11")
@@
     (pin "19")
     (pin "2")
-    (pin "2")
     (pin "20")
     (pin "21")
@@
     (pin "9")
   )
+  (symbol (lib_id "symbols:PinLengths") (at 67.31 147.32 0) (unit 1)
+    (in_bom yes) (on_board yes) (fields_autoplaced)
+    (property "Reference" "U7" (id 0) (at 63.5 137.16 0))
+    (property "Value" "" (id 1) (at 63.5 139.7 0))
+    (property "Footprint" "" (id 2) (at 55.245 135.89 0)
+      (effects (font (size 1.27 1.27)) hide)
+    )
+    (property "Datasheet" "" (id 3) (at 55.245 135.89 0)
+      (effects (font (size 1.27 1.27)) hide)
+    )
+    (pin "1")
+    (pin "2")
+    (pin "3")
+    (pin "4")
+    (pin "5")
+    (pin "6")
+  )
   (symbol (lib_id "symbols:PinCushion") (at 144.78 170.18 0) (unit 1)
     (in_bom yes) (on_board yes) (fields_autoplaced)
@@
       (effects (font (size 1.27 1.27)) hide)
     )
+    (pin "1")
     (pin "10")
     (pin "11")
@@
     (pin "19")
     (pin "2")
-    (pin "2")
     (pin "20")
     (pin "21")
@@
     (pin "9")
   )
+  (symbol (lib_name "PinLengths_3") (lib_id "symbols:PinLengths") (at 95.25 177.165 270) (unit 1)
+    (in_bom yes) (on_board yes) (fields_autoplaced)
+    (property "Reference" "U9" (id 0) (at 100.965 172.0849 90)
+      (effects (font (size 1.27 1.27)) (justify left))
+    )
+    (property "Value" "" (id 1) (at 100.965 174.6249 90)
+      (effects (font (size 1.27 1.27)) (justify left))
+    )
+    (property "Footprint" "" (id 2) (at 106.68 165.1 0)
+      (effects (font (size 1.27 1.27)) hide)
+    )
+    (property "Datasheet" "" (id 3) (at 106.68 165.1 0)
+      (effects (font (size 1.27 1.27)) hide)
+    )
+    (pin "1")
+    (pin "2")
+    (pin "3")
+    (pin "4")
+    (pin "5")
+    (pin "6")
+  )
+  (symbol (lib_name "PinLengths_2") (lib_id "symbols:PinLengths") (at 85.09 146.685 90) (unit 1)
+    (in_bom yes) (on_board yes) (fields_autoplaced)
+    (property "Reference" "U8" (id 0) (at 99.695 149.2249 90)
+      (effects (font (size 1.27 1.27)) (justify right))
+    )
+    (property "Value" "" (id 1) (at 99.695 151.7649 90)
+      (effects (font (size 1.27 1.27)) (justify right))
+    )
+    (property "Footprint" "" (id 2) (at 73.66 158.75 0)
+      (effects (font (size 1.27 1.27)) hide)
+    )
+    (property "Datasheet" "" (id 3) (at 73.66 158.75 0)
+      (effects (font (size 1.27 1.27)) hide)
+    )
+    (pin "1")
+    (pin "2")
+    (pin "3")
+    (pin "4")
+    (pin "5")
+    (pin "6")
+  )
+  (symbol (lib_name "PinLengths_4") (lib_id "symbols:PinLengths") (at 59.69 179.705 180) (unit 1)
+    (in_bom yes) (on_board yes) (fields_autoplaced)
+    (property "Reference" "U6" (id 0) (at 70.485 173.9899 0)
+      (effects (font (size 1.27 1.27)) (justify right))
+    )
+    (property "Value" "" (id 1) (at 70.485 176.5299 0)
+      (effects (font (size 1.27 1.27)) (justify right))
+    )
+    (property "Footprint" "" (id 2) (at 71.755 191.135 0)
+      (effects (font (size 1.27 1.27)) hide)
+    )
+    (property "Datasheet" "" (id 3) (at 71.755 191.135 0)
+      (effects (font (size 1.27 1.27)) hide)
+    )
+    (pin "1")
+    (pin "2")
+    (pin "3")
+    (pin "4")
+    (pin "5")
+    (pin "6")
+  )
   (sheet_instances
     (path "/" (page "1"))
@@
       (reference "U5") (unit 1) (value "PinCushion") (footprint "")
     )
-  )
+    (path "/f5c00da9-489a-4e67-a4b6-d36281634477"
+      (reference "U6") (unit 1) (value "PinLengths") (footprint "")
+    )
+    (path "/b851059d-e341-4edc-b150-88f2b168e573"
+      (reference "U7") (unit 1) (value "PinLengths") (footprint "")
+    )
+    (path "/f5a9aa21-6ccc-4e3e-89d0-121d5266727a"
+      (reference "U8") (unit 1) (value "PinLengths") (footprint "")
+    )
+    (path "/f1aeb88f-5f89-4537-86d8-f06e86582872"
+      (reference "U9") (unit 1) (value "PinLengths") (footprint "")
+    )
+    (path "/415878dc-1d5e-448e-8e04-df0e5d096ef7"
+      (reference "U?") (unit 1) (value "PinLengths") (footprint "")
+    )
+    (path "/5271bf79-264b-4a63-8389-35fabf857755"
+      (reference "U?") (unit 1) (value "PinLengths") (footprint "")
+    )
+    (path "/96536b7b-7f39-4027-a516-d77fe63257c0"
+      (reference "U?") (unit 1) (value "PinLengths") (footprint "")
+    )
+  )

Commit message: update annotations
Parts:
- gave numbers to parts that had none: 3
Changed lines of the file:
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@@
   (symbol (lib_id "symbols:PinLengths") (at 194.945 149.86 0) (mirror x) (unit 1)
     (in_bom yes) (on_board yes) (fields_autoplaced)
-    (property "Reference" "U?" (id 0) (at 191.135 160.02 0))
+    (property "Reference" "U11" (id 0) (at 191.135 160.02 0))
     (property "Value" "" (id 1) (at 191.135 157.48 0))
     (property "Footprint" "" (id 2) (at 182.88 161.29 0)
@@
   (symbol (lib_name "PinLengths_1") (lib_id "symbols:PinLengths") (at 110.49 132.08 90) (unit 1)
     (in_bom yes) (on_board yes) (fields_autoplaced)
-    (property "Reference" "U?" (id 0) (at 125.095 134.6199 90)
+    (property "Reference" "U10" (id 0) (at 125.095 134.6199 90)
       (effects (font (size 1.27 1.27)) (justify right))
     )
@@
   (symbol (lib_id "symbols:PinLengths") (at 222.885 142.24 0) (mirror y) (unit 1)
     (in_bom yes) (on_board yes) (fields_autoplaced)
-    (property "Reference" "U?" (id 0) (at 226.695 132.08 0))
+    (property "Reference" "U12" (id 0) (at 226.695 132.08 0))
     (property "Value" "" (id 1) (at 226.695 134.62 0))
     (property "Footprint" "" (id 2) (at 234.95 130.81 0)
@@
       (reference "U9") (unit 1) (value "PinLengths") (footprint "")
     )
+    (path "/5271bf79-264b-4a63-8389-35fabf857755"
+      (reference "U10") (unit 1) (value "PinLengths") (footprint "")
+    )
     (path "/415878dc-1d5e-448e-8e04-df0e5d096ef7"
-      (reference "U?") (unit 1) (value "PinLengths") (footprint "")
-    )
-    (path "/5271bf79-264b-4a63-8389-35fabf857755"
-      (reference "U?") (unit 1) (value "PinLengths") (footprint "")
+      (reference "U11") (unit 1) (value "PinLengths") (footprint "")
     )
     (path "/96536b7b-7f39-4027-a516-d77fe63257c0"
-      (reference "U?") (unit 1) (value "PinLengths") (footprint "")
-    )
-  )
+      (reference "U12") (unit 1) (value "PinLengths") (footprint "")
+    )
+  )
